File: pcb/pcb/components.kicad_sch (KiCad schematic)
At the start: 11 parts, among them J10 Mic, J11 Mic, J5 Micro SD Card, J6 SD Card, J7 Relay Solenoid, J8 Power, J9 Status LED, K1 Relay

Commit message: update pcd mit Notöffnung
Parts:
- added SW6: Notöffnung, symbol Switch:SW_Push
Connections:
- net at J8.1 (12V), K1.7, K1.8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: now also SW6.1
- net at K1.1, K1.14, L1.1 (-): now also SW6.2
Other:
- title: (none) -> Externe Komponenten
- moved on the sheet: D2
