File: pcb/pcb/components.kicad_sch (KiCad schematic)
At the start: 12 parts, among them J10 Mic, J11 Mic, J5 Micro SD Card, J6 SD Card, J7 Relay Solenoid, J8 Power, J9 Status LED, K1 Relay, SW6 Notöffnung

Commit message: update pcb
Parts:
- SW6: footprint (none) -> Button_Switch_SMD:SW_SPST_Omron_B3FS-101xP
Changed lines of the file:
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@@
 			)
 		)
-		(property "Footprint" ""
+		(property "Footprint" "Button_Switch_SMD:SW_SPST_Omron_B3FS-101xP"
 			(at 82.55 76.2 0)
 			(effects

Commit message: update
Parts:
- K1: footprint Relay_THT:Relay_StandexMeder_DIP_LowProfile -> (none)
- PS1: footprint Converter_DCDC:Converter_DCDC_XP_POWER-IAxxxxD_THT -> (none)
Changed lines of the file:
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@@
 			)
 		)
-		(property "Footprint" "Converter_DCDC:Converter_DCDC_XP_POWER-IAxxxxD_THT"
+		(property "Footprint" ""
 			(at 21.59 132.08 0)
 			(effects
@@
 			)
 		)
-		(property "Footprint" "Relay_THT:Relay_StandexMeder_DIP_LowProfile"
+		(property "Footprint" ""
 			(at 83.82 109.22 0)
 			(effects

Commit message: Final_PCB
Parts:
- J10, J11: footprint (none) -> TerminalBlock:TerminalBlock_MaiXu_MX126-5.0-04P_1x04_P5.00mm
- J5, J6, PS1: footprint (none) -> TerminalBlock:TerminalBlock_MaiXu_MX126-5.0-06P_1x06_P5.00mm
- J7, J9, K1, L1: footprint (none) -> TerminalBlock:TerminalBlock_bornier-3_P5.08mm
- J8: footprint (none) -> TerminalBlock:TerminalBlock_bornier-2_P5.08mm
- SW6: footprint Button_Switch_SMD:SW_SPST_Omron_B3FS-101xP -> Button_Switch_THT:SW_PUSH_6mm_H4.3mm
Changed lines of the file:
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@@
 			)
 		)
-		(property "Footprint" ""
+		(property "Footprint" "TerminalBlock:TerminalBlock_bornier-2_P5.08mm"
 			(at 19.05 124.46 0)
 			(effects
@@
 			)
 		)
-		(property "Footprint" ""
+		(property "Footprint" "TerminalBlock:TerminalBlock_MaiXu_MX126-5.0-04P_1x04_P5.00mm"
 			(at 53.34 176.53 0)
 			(effects
@@
 			)
 		)
-		(property "Footprint" ""
+		(property "Footprint" "TerminalBlock:TerminalBlock_bornier-3_P5.08mm"
 			(at 24.13 97.79 0)
 			(effects
@@
 			)
 		)
-		(property "Footprint" ""
+		(property "Footprint" "TerminalBlock:TerminalBlock_bornier-3_P5.08mm"
 			(at 104.775 114.3 90)
 			(effects
@@
 			)
 		)
-		(property "Footprint" ""
+		(property "Footprint" "TerminalBlock:TerminalBlock_MaiXu_MX126-5.0-06P_1x06_P5.00mm"
 			(at 107.95 30.48 0)
 			(effects
@@
 			)
 		)
-		(property "Footprint" ""
+		(property "Footprint" "TerminalBlock:TerminalBlock_MaiXu_MX126-5.0-06P_1x06_P5.00mm"
 			(at 21.59 132.08 0)
 			(effects
@@
 			)
 		)
-		(property "Footprint" ""
+		(property "Footprint" "TerminalBlock:TerminalBlock_bornier-3_P5.08mm"
 			(at 83.82 109.22 0)
 			(effects
@@
 			)
 		)
-		(property "Footprint" ""
+		(property "Footprint" "TerminalBlock:TerminalBlock_MaiXu_MX126-5.0-06P_1x06_P5.00mm"
 			(at 22.86 35.56 0)
 			(effects
@@
 			)
 		)
-		(property "Footprint" "Button_Switch_SMD:SW_SPST_Omron_B3FS-101xP"
+		(property "Footprint" "Button_Switch_THT:SW_PUSH_6mm_H4.3mm"
 			(at 82.55 76.2 0)
 			(effects
@@
 			)
 		)
-		(property "Footprint" ""
+		(property "Footprint" "TerminalBlock:TerminalBlock_bornier-3_P5.08mm"
 			(at 21.59 156.21 0)
 			(effects
@@
 			)
 		)
-		(property "Footprint" ""
+		(property "Footprint" "TerminalBlock:TerminalBlock_MaiXu_MX126-5.0-04P_1x04_P5.00mm"
 			(at 20.32 176.53 0)
 			(effects

Commit message: PCB update
Parts:
- D2: footprint LED_SMD:LED_WS2812B_PLCC4_5.0x5.0mm_P3.2mm -> (none)
- J10, J11: footprint TerminalBlock:TerminalBlock_MaiXu_MX126-5.0-04P_1x04_P5.00mm -> (none)
- J5, J6, PS1: footprint TerminalBlock:TerminalBlock_MaiXu_MX126-5.0-06P_1x06_P5.00mm -> (none)
- J7, J9, K1, L1: footprint TerminalBlock:TerminalBlock_bornier-3_P5.08mm -> (none)
- J8: footprint TerminalBlock:TerminalBlock_bornier-2_P5.08mm -> (none)
- SW6: footprint Button_Switch_THT:SW_PUSH_6mm_H4.3mm -> (none)
Changed lines of the file:
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@@
 			)
 		)
-		(property "Footprint" "TerminalBlock:TerminalBlock_bornier-2_P5.08mm"
+		(property "Footprint" ""
 			(at 19.05 124.46 0)
 			(effects
@@
 			)
 		)
-		(property "Footprint" "TerminalBlock:TerminalBlock_MaiXu_MX126-5.0-04P_1x04_P5.00mm"
+		(property "Footprint" ""
 			(at 53.34 176.53 0)
 			(effects
@@
 			)
 		)
-		(property "Footprint" "TerminalBlock:TerminalBlock_bornier-3_P5.08mm"
+		(property "Footprint" ""
 			(at 24.13 97.79 0)
 			(effects
@@
 			)
 		)
-		(property "Footprint" "TerminalBlock:TerminalBlock_bornier-3_P5.08mm"
+		(property "Footprint" ""
 			(at 104.775 114.3 90)
 			(effects
@@
 			)
 		)
-		(property "Footprint" "TerminalBlock:TerminalBlock_MaiXu_MX126-5.0-06P_1x06_P5.00mm"
+		(property "Footprint" ""
 			(at 107.95 30.48 0)
 			(effects
@@
 			)
 		)
-		(property "Footprint" "TerminalBlock:TerminalBlock_MaiXu_MX126-5.0-06P_1x06_P5.00mm"
+		(property "Footprint" ""
 			(at 21.59 132.08 0)
 			(effects
@@
 			)
 		)
-		(property "Footprint" "TerminalBlock:TerminalBlock_bornier-3_P5.08mm"
+		(property "Footprint" ""
 			(at 83.82 109.22 0)
 			(effects
@@
 			)
 		)
-		(property "Footprint" "TerminalBlock:TerminalBlock_MaiXu_MX126-5.0-06P_1x06_P5.00mm"
+		(property "Footprint" ""
 			(at 22.86 35.56 0)
 			(effects
@@
 			)
 		)
-		(property "Footprint" "Button_Switch_THT:SW_PUSH_6mm_H4.3mm"
+		(property "Footprint" ""
 			(at 82.55 76.2 0)
 			(effects
@@
 			)
 		)
-		(property "Footprint" "LED_SMD:LED_WS2812B_PLCC4_5.0x5.0mm_P3.2mm"
+		(property "Footprint" ""
 			(at 87.63 161.29 0)
 			(effects
@@
 			)
 		)
-		(property "Footprint" "TerminalBlock:TerminalBlock_bornier-3_P5.08mm"
+		(property "Footprint" ""
 			(at 21.59 156.21 0)
 			(effects
@@
 			)
 		)
-		(property "Footprint" "TerminalBlock:TerminalBlock_MaiXu_MX126-5.0-04P_1x04_P5.00mm"
+		(property "Footprint" ""
 			(at 20.32 176.53 0)
 			(effects
