File: pcb/pcb/pcb.kicad_pcb (KiCad board)
At the start: 2 copper layers, 1 part

Commit message: PCB update
Parts:
- removed the REF** at (112.6, 78.2)
- added C1: 47nF, Capacitor_THT:C_Disc_D5.0mm_W2.5mm_P5.00mm, F.Cu at (136.5, 126.0)
- added C2: 47nF, Capacitor_THT:C_Disc_D5.0mm_W2.5mm_P5.00mm, F.Cu at (152.0, 126.0)
- added C3: 47nF, Capacitor_THT:C_Disc_D5.0mm_W2.5mm_P5.00mm, F.Cu at (167.5, 126.0)
- added C4: 47nF, Capacitor_THT:C_Disc_D5.0mm_W2.5mm_P5.00mm, F.Cu at (181.5, 126.0)
- added C5: 47nF, Capacitor_THT:C_Disc_D5.0mm_W2.5mm_P5.00mm, F.Cu at (196.5, 126.0)
- added D1: WS2812B, LED_SMD:LED_WS2812B_PLCC4_5.0x5.0mm_P3.2mm, F.Cu at (197.1, 79.8)
- added D3: WS2812B, LED_SMD:LED_WS2812B_PLCC4_5.0x5.0mm_P3.2mm, F.Cu at (184.1, 79.8)
- added J1: SD Card, TerminalBlock:TerminalBlock_MaiXu_MX126-5.0-06P_1x06_P5.00mm, F.Cu at (96.5, 65.0)
- added J2: Mic, TerminalBlock:TerminalBlock_MaiXu_MX126-5.0-04P_1x04_P5.00mm, F.Cu at (131.0, 65.0)
- added J3: Relay Solenoid, TerminalBlock:TerminalBlock_bornier-3_P5.08mm, F.Cu at (168.3, 64.5)
- added J4: Status LED, TerminalBlock:TerminalBlock_bornier-3_P5.08mm, F.Cu at (188.3, 64.5)
- added P1: Power, TerminalBlock:TerminalBlock_bornier-2_P5.08mm, F.Cu at (154.5, 65.0)
- added R1: 1kΩ, Resistor_THT:R_Axial_DIN0207_L6.3mm_D2.5mm_P10.16mm_Horizontal, F.Cu at (136.0, 117.4)
- added R10: 1kΩ, Resistor_THT:R_Axial_DIN0207_L6.3mm_D2.5mm_P10.16mm_Horizontal, F.Cu at (201.5, 117.5)
- added R2: 10kΩ, Resistor_THT:R_Axial_DIN0207_L6.3mm_D2.5mm_P10.16mm_Horizontal, F.Cu at (142.5, 117.4)
- added R3: 10kΩ, Resistor_THT:R_Axial_DIN0207_L6.3mm_D2.5mm_P10.16mm_Horizontal, F.Cu at (151.7, 117.4)
- added R4: 1kΩ, Resistor_THT:R_Axial_DIN0207_L6.3mm_D2.5mm_P10.16mm_Horizontal, F.Cu at (157.4, 117.4)
- added R5: 10kΩ, Resistor_THT:R_Axial_DIN0207_L6.3mm_D2.5mm_P10.16mm_Horizontal, F.Cu at (166.8, 117.4)
- added R6: 1kΩ, Resistor_THT:R_Axial_DIN0207_L6.3mm_D2.5mm_P10.16mm_Horizontal, F.Cu at (172.5, 117.4)
- added R7: 10kΩ, Resistor_THT:R_Axial_DIN0207_L6.3mm_D2.5mm_P10.16mm_Horizontal, F.Cu at (180.8, 117.4)
- added R8: 1kΩ, Resistor_THT:R_Axial_DIN0207_L6.3mm_D2.5mm_P10.16mm_Horizontal, F.Cu at (187.0, 117.5)
- added R9: 10kΩ, Resistor_THT:R_Axial_DIN0207_L6.3mm_D2.5mm_P10.16mm_Horizontal, F.Cu at (195.4, 117.5)
- added REF**: XCVR_ESP32-C3_DEVKITC-02, footprints:XCVR_ESP32-C3-DEVKITC-02, F.Cu at (108.1, 108.3)
- added SW1: Button Up, Button_Switch_THT:SW_PUSH_6mm_H4.3mm, F.Cu at (136.0, 93.3)
- added SW2: Button Down, Button_Switch_THT:SW_PUSH_6mm_H4.3mm, F.Cu at (151.0, 93.5)
- added SW3: Button Record, Button_Switch_THT:SW_PUSH_6mm_H4.3mm, F.Cu at (166.5, 93.5)
- added SW4: Button Delete, Button_Switch_THT:SW_PUSH_6mm_H4.3mm, F.Cu at (180.5, 93.5)
- added SW5: Button Play, Button_Switch_THT:SW_PUSH_6mm_H4.3mm, F.Cu at (195.0, 93.5)
Routing:
- net 5V: track 0.00 -> 411.0 mm
- net GND: track 0.00 -> 145.3 mm
- net Net-(J1-MOSI): track 0.00 -> 64.6 mm
- net Net-(J1-CS): track 0.00 -> 55.2 mm
- net Net-(J1-SCK): track 0.00 -> 48.4 mm
- net Net-(J1-MISO): track 0.00 -> 47.3 mm
- net Net-(J2-A0): track 0.00 -> 33.2 mm

Commit message: verkabelung fertig
Parts:
- moved D1 86.6 mm to (110.5, 84.7), turned to 180 degrees
- moved R10 70.1 mm to (132.2, 106.8), turned to -90 degrees
- moved SW5 63.2 mm to (131.8, 93.5)
- moved C5 58.8 mm to (137.8, 126.0), turned to 180 degrees
- moved R9 58.2 mm to (138.2, 106.8), turned to -90 degrees
- moved R3 47.5 mm to (197.8, 106.5), turned to -90 degrees
- moved C1 46.0 mm to (182.5, 126.5), turned to 180 degrees
- moved C2 45.5 mm to (197.5, 126.5), turned to 180 degrees
- moved R1 42.8 mm to (177.5, 107.0), turned to -90 degrees
- moved R2 41.8 mm to (183.0, 106.9), turned to -90 degrees
- moved SW1 40.5 mm to (176.5, 93.5)
- moved SW2 40.5 mm to (191.5, 93.5)
- moved R4 36.4 mm to (192.1, 106.5), turned to -90 degrees
- moved R8 27.4 mm to (161.9, 106.3), turned to -90 degrees
- moved R6 26.8 mm to (148.1, 106.4), turned to -90 degrees
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Routing:
- net GND: track 145.3 -> 302.0 mm
- net Net-(U1-GPIO1): track 0.00 -> 96.9 mm
- net Net-(U1-GPIO2): track 0.00 -> 80.8 mm
- net Net-(D1-DOUT): track 0.00 -> 79.0 mm
- net Net-(U1-GPIO9): track 0.00 -> 68.9 mm
- net 5V: track 411.0 -> 475.6 mm
- net Net-(U1-GPIO10): track 0.00 -> 62.2 mm
- net Net-(D1-DIN): track 0.00 -> 34.8 mm
- net Net-(U1-GPIO19/USBD_+): track 0.00 -> 31.1 mm
- net Net-(R10-Pad1): track 0.00 -> 21.4 mm
- net Net-(R7-Pad1): track 0.00 -> 21.2 mm
- net Net-(R1-Pad1): track 0.00 -> 21.0 mm
- net Net-(R3-Pad1): track 0.00 -> 20.8 mm
- net Net-(R5-Pad1): track 0.00 -> 20.8 mm
- net Net-(D3-DOUT): track 0.00 -> 15.7 mm
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
Commit message: PCB Update
Parts:
- moved D1 6.50 mm to (110.5, 78.2)
Routing:
- net Net-(D1-DIN): track 34.8 -> 41.3 mm
- net 5V: track 475.6 -> 482.1 mm
- net GND: track 302.0 -> 306.5 mm
- net Net-(D1-DOUT): track 79.0 -> 83.4 mm
Changed lines of the file:
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@@
 	(footprint "LED_SMD:LED_WS2812B_PLCC4_5.0x5.0mm_P3.2mm"
 		(layer "F.Cu")
-		(at 110.55 84.65 180)
+		(at 110.55 78.15 180)
 		(descr "5.0mm x 5.0mm Addressable RGB LED NeoPixel, https://cdn-shop.adafruit.com/datasheets/WS2812B.pdf")
 		(tags "LED RGB NeoPixel PLCC-4 5050")
@@
 	(segment
 		(start 104.58 83)
+		(end 104.54 83.04)
+		(width 0.2)
+		(layer "F.Cu")
+		(net 2)
+	)
+	(segment
+		(start 104.54 83.04)
+		(end 104.54 80.06)
+		(width 0.2)
+		(layer "F.Cu")
+		(net 2)
+	)
+	(segment
+		(start 104.54 83.04)
 		(end 96.64 90.94)
+		(width 0.2)
+		(layer "F.Cu")
+		(net 2)
+	)
+	(segment
+		(start 104.54 80.06)
+		(end 108.1 76.5)
 		(width 0.2)
 		(layer "F.Cu")
@@
 	)
 	(segment
-		(start 108.1 83)
-		(end 104.58 83)
-		(width 0.2)
-		(layer "F.Cu")
-		(net 2)
-	)
-	(segment
 		(start 133.85 127.1)
 		(end 132.75 126)
@@
 	)
 	(segment
-		(start 108.1 86.3)
+		(start 108.1 79.8)
 		(end 108.1 104.88)
 		(width 0.2)
 		(layer "F.Cu")
 		(net 7)
+	)
+	(segment
+		(start 116.5 83)
+		(end 116.5 80)
+		(width 0.2)
+		(layer "F.Cu")
+		(net 8)
+	)
+	(segment
+		(start 116.5 83)
+		(end 189 83)
+		(width 0.2)
+		(layer "F.Cu")
+		(net 8)
 	)
 	(segment
@@
 	)
 	(segment
+		(start 116.5 80)
+		(end 113 76.5)
+		(width 0.2)
+		(layer "F.Cu")
+		(net 8)
+	)
+	(segment
 		(start 189 83)
 		(end 190 82)
@@
 	)
 	(segment
-		(start 113 83)
-		(end 189 83)
-		(width 0.2)
-		(layer "F.Cu")
-		(net 8)
-	)
-	(segment
 		(start 198 85.1)
 		(end 198 93.5)
@@
 	)
 	(segment
-		(start 113 86.3)
-		(end 113 105.06)
-		(width 0.2)
-		(layer "F.Cu")
-		(net 9)
-	)
-	(segment
 		(start 194.9 82)
 		(end 198 85.1)
@@
 		(width 0.2)
 		(layer "F.Cu")
+		(net 9)
+	)
+	(segment
+		(start 113 79.8)
+		(end 113 105.06)
+		(width 0.2)
+		(layer "F.Cu")

Commit message: PCB-Update
Parts:
- moved J1 43.0 mm to (80.4, 104.9), turned to 90 degrees
- moved J2 37.1 mm to (93.9, 64.4)
- moved P1 25.7 mm to (128.8, 63.9)
- moved D1 20.5 mm to (130.9, 80.2)
- moved J3 13.9 mm to (154.5, 63.9)
- moved D3 2.50 mm to (194.9, 80.2)
- moved C3 1.77 mm to (152.4, 126.4)
- moved C4 1.77 mm to (166.4, 126.4)
- moved R1 1.29 mm to (176.4, 106.3)
- moved R2 1.29 mm to (181.9, 106.2)
- moved R10 1.25 mm to (131.1, 106.2)
- moved R9 1.25 mm to (137.2, 106.2)
- moved C5 1.17 mm to (136.7, 126.4)
- moved R5 1.10 mm to (152.8, 106.3)
- moved R6 1.10 mm to (147.0, 106.3)
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Routing:
- net 5V: track 482.1 -> 385.3 mm
- net Net-(J1-CS): track 55.2 -> 19.2 mm
- net GND: track 306.5 -> 339.5 mm
- net Net-(J1-MOSI): track 64.6 -> 33.0 mm
- net Net-(J1-SCK): track 48.4 -> 17.1 mm
- net Net-(D1-DOUT): track 83.4 -> 60.5 mm
- net Net-(J1-MISO): track 47.3 -> 33.1 mm
- net Net-(D1-DIN): track 41.3 -> 52.8 mm
- net Net-(J2-A0): track 33.2 -> 39.8 mm
- net Net-(U1-GPIO19/USBD_+): track 31.1 -> 32.9 mm
- net Net-(D3-DOUT): track 15.7 -> 14.2 mm
- net Net-(U1-GPIO9): track 68.9 -> 70.2 mm
- net Net-(U1-GPIO10): track 62.2 -> 63.1 mm
- net Net-(R1-Pad1): track 21.0 -> 20.4 mm
- net (no net): track 0.51 -> 0.00 mm
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Other:
- board outline added: 150 x 90 mm
- board text added: "Button Delete"
- board text added: "Button Down"
- board text added: "Button Play"
- board text added: "Button Record"
- board text added: "Button Up"
- board text added: "LED"
- board text added: "Mic"
- board text added: "Power"
- board text added: "Relay"
- board text added: "SD Card"
- board text added: "Status LED"

Commit message: update
Parts:
- added G***: LOGO, New_Library:QR_Code_10-10, F.Cu at (75.0, 118.5)
- added G***: LOGO, New_Library:HN_FB03_Logo_komplett_50mm, F.Cu at (160.0, 81.0)
- moved C1 4.55 mm to (178.2, 123.2)
- moved C2 4.55 mm to (193.2, 123.2)
- moved C3 4.55 mm to (149.2, 123.2)
- moved C4 4.55 mm to (163.2, 123.2)
- moved C5 4.55 mm to (133.4, 123.2)
- moved J1 4.55 mm to (77.2, 101.7)
- moved J2 4.55 mm to (90.7, 61.2)
- moved J4 4.55 mm to (184.0, 61.2)
- moved R3 4.55 mm to (193.5, 103.2)
- moved R4 4.55 mm to (187.8, 103.2)
- moved R5 4.55 mm to (149.5, 103.1)
- moved R6 4.55 mm to (143.8, 103.1)
- moved R7 4.55 mm to (163.8, 103.1)
- moved R8 4.55 mm to (157.6, 103.0)
- moved REF** 4.55 mm to (103.8, 105.0)
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Other:
- board size 150 x 90 mm -> 140 x 80 mm
- board text added: "LED Status"
- board text removed: "LED"

Commit message: Finale_PCB???
Parts:
- moved G*** 2.24 mm to (77.0, 117.5)
- moved G*** 1.00 mm to (161.0, 81.0)
Other:
- board size 140 x 80 mm -> 135 x 80 mm

Commit message: NochmalFinal
Parts:
- moved G*** 1.80 mm to (78.5, 118.5)
Other:
- board size 135 x 80 mm -> 130 x 80 mm
Changed lines of the file:
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@@
 	(footprint "New_Library:QR_Code_10-10"
 		(layer "F.Cu")
-		(at 77 117.5)
+		(at 78.5 118.5)
 		(property "Reference" "G***"
 			(at 0 0 0)
@@
 	)
 	(gr_rect
-		(start 66 50.5)
-		(end 201 130.5)
+		(start 70 50.5)
+		(end 200 130.5)
 		(stroke
 			(width 0.2)
@@
 	)
 	(gr_text "SD Card"
-		(at 70.285 95.785 90)
+		(at 85 97.5 90)
 		(layer "F.SilkS")
 		(effects
@@
 		(layer "User.1")
 		(pts
-			(xy 201 50.5) (xy 201 130.5)
+			(xy 70 130.5) (xy 200 130.5)
 		)
-		(height -11.5)
-		(gr_text "80,0000 mm"
-			(at 210.7 90.5 90)
+		(height 7.5)
+		(gr_text "130,0000 mm"
+			(at 135 136.2 0)
 			(layer "User.1")
 			(effects
@@
 		(layer "User.1")
 		(pts
-			(xy 66 130.5) (xy 201 130.5)
+			(xy 200 50.5) (xy 200 130.5)
 		)
-		(height 9.5)
-		(gr_text "135,0000 mm"
-			(at 133.5 138.2 0)
+		(height -13)
+		(gr_text "80,0000 mm"
+			(at 211.2 90.5 90)
 			(layer "User.1")
 			(effects

Commit message: Finish 100x80
Parts:
- G***: moved to B.Cu
- moved J1 62.2 mm to (134.5, 77.5), turned to 0 degrees
- moved G*** 58.4 mm to (114.5, 72.5)
- moved D1 46.9 mm to (174.6, 77.9)
- moved J2 20.8 mm to (111.3, 58.5)
- moved G*** 15.9 mm to (171.5, 69.0), turned to 180 degrees
- moved P1 11.9 mm to (137.2, 58.3)
- moved REF** 11.8 mm to (115.6, 105.8)
- moved SW5 6.07 mm to (133.5, 90.0)
- moved J4 5.86 mm to (178.8, 58.5)
- moved J3 5.57 mm to (156.3, 58.3)
- moved C5 5.57 mm to (139.0, 123.0)
- moved R9 5.57 mm to (139.5, 102.8)
- moved R10 5.57 mm to (133.4, 102.8)
- moved C3 5.47 mm to (154.7, 123.2)
- moved R5 5.47 mm to (155.0, 103.1)
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Routing:
- net Net-(D1-DOUT): track 60.5 -> 10.5 mm
- net Net-(D1-DIN): track 52.8 -> 94.7 mm
- net Net-(J1-CS): track 19.2 -> 58.6 mm
- net Net-(J2-A0): track 39.8 -> 78.6 mm
- net Net-(J1-SCK): track 17.1 -> 48.2 mm
- net Net-(J1-MISO): track 33.1 -> 62.9 mm
- net GND: track 339.5 -> 363.2 mm
- net 5V: track 385.3 -> 407.9 mm
- net Net-(J1-MOSI): track 33.0 -> 52.2 mm
- net Net-(U1-GPIO9): track 70.2 -> 64.0 mm
- net Net-(U1-GPIO10): track 63.1 -> 57.0 mm
- net Net-(D3-DOUT): track 14.2 -> 20.3 mm
- net Net-(U1-GPIO19/USBD_+): track 32.9 -> 27.4 mm
- net Net-(U1-GPIO1): track 97.4 -> 93.5 mm
- net Net-(U1-GPIO2): track 81.1 -> 78.7 mm
Other:
- board size 130 x 80 mm -> 100 x 80 mm
- board text added: "Group 9"
- board text added: "Klopf - Klopf"
- board text added: "Piezo"
- board text removed: "Mic"
