File: pcb/pcb/pcb.kicad_pcb (KiCad board)
At the start: 2 copper layers, 100 x 80 mm, 30 parts, among them J1 SD Card, J2 Mic, J3 Relay Solenoid, J4 Status LED, P1 Power, SW1 Button Up, SW2 Button Down, SW3 Button Record, SW4 Button Delete, SW5 Button Play

Commit message: Finish
Parts:
- moved J1 4.03 mm to (138.0, 79.5)
- moved C1 2.23 mm to (183.0, 125.4)
- moved C2 2.23 mm to (195.9, 125.4)
- moved C3 2.23 mm to (154.7, 125.4)
- moved C4 2.23 mm to (168.4, 125.4)
- moved C5 2.23 mm to (139.0, 125.2)
- moved R1 2.23 mm to (178.0, 105.3)
- moved R10 2.23 mm to (133.4, 105.1)
- moved R2 2.23 mm to (183.5, 105.3)
- moved R3 2.23 mm to (196.2, 105.4)
- moved R4 2.23 mm to (190.5, 105.4)
- moved R5 2.23 mm to (155.0, 105.3)
- moved R6 2.23 mm to (149.2, 105.3)
- moved R7 2.23 mm to (169.0, 105.3)
- moved R8 2.23 mm to (162.8, 105.2)
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Routing:
- net Net-(J2-A0): track 78.6 -> 86.8 mm
- net 5V: track 407.9 -> 413.0 mm
- net GND: track 363.2 -> 367.6 mm
- net Net-(J1-SCK): track 48.2 -> 50.9 mm
- net Net-(J1-MOSI): track 52.2 -> 54.9 mm
- net Net-(J1-CS): track 58.6 -> 61.3 mm
- net Net-(U1-GPIO2): track 78.7 -> 81.0 mm
- net Net-(U1-GPIO10): track 57.0 -> 59.2 mm
- net Net-(U1-GPIO1): track 93.5 -> 95.8 mm
- net Net-(U1-GPIO19/USBD_+): track 27.4 -> 26.4 mm
- net Net-(U1-GPIO9): track 64.0 -> 63.1 mm

Commit message: Finally
Routing:
- net Net-(J2-A0): track 86.8 -> 88.7 mm
Changed lines of the file:
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@@
-	)
-	(segment
-		(start 155 82)
-		(end 155 79.095836)
-		(width 0.2)
-		(layer "B.Cu")
-		(net 15)
 	)
 	(segment
@@
 	)
 	(segment
-		(start 148.5 88.5)
-		(end 155 82)
+		(start 155.5 81.5)
+		(end 155.5 77)
 		(width 0.2)
 		(layer "B.Cu")
@@
 	)
 	(segment
-		(start 155 79.095836)
-		(end 137.804164 61.9)
+		(start 155.5 77)
+		(end 140.4 61.9)
 		(width 0.2)
 		(layer "B.Cu")
@@
 	)
 	(segment
-		(start 137.804164 61.9)
+		(start 148.5 88.5)
+		(end 155.5 81.5)
+		(width 0.2)
+		(layer "B.Cu")
+		(net 15)
+	)
+	(segment
+		(start 140.4 61.9)
 		(end 114.715 61.9)
 		(width 0.2)

Commit message: Change PCB/TEST
Parts:
- removed SW5: Button Play, Button_Switch_THT:SW_PUSH_6mm_H4.3mm
Routing:
- net 5V: track 413.0 -> 397.1 mm
- net Net-(R10-Pad1): track 20.9 -> 14.4 mm
Other:
- board text removed: "Button Play"

Commit message: Finale Change PCB
Parts:
- removed C5: 47nF, Capacitor_THT:C_Disc_D5.0mm_W2.5mm_P5.00mm
- removed R10: 1kΩ, Resistor_THT:R_Axial_DIN0207_L6.3mm_D2.5mm_P10.16mm_Horizontal
- removed R9: 10kΩ, Resistor_THT:R_Axial_DIN0207_L6.3mm_D2.5mm_P10.16mm_Horizontal
- U1: renamed from REF**; value XCVR_ESP32-C3_DEVKITC-02 -> ESP32-C3-DevKitC-02
- moved C3 1.85 mm to (156.5, 125.5)
- moved R5 1.50 mm to (156.5, 105.4)
- moved C4 1.10 mm to (169.5, 125.5)
- moved R6 0.77 mm to (150.0, 105.5)
- moved SW3 0.77 mm to (150.0, 92.5)
- moved R7 0.53 mm to (169.5, 105.5)
- moved R8 0.30 mm to (163.0, 105.5)
- moved SW4 0.18 mm to (163.0, 92.5)
Connections:
- C3 pad 1: Net-(U1-GPIO9) -> Net-(U1-GPIO18/USBD_-)
- J3 pad 3: GND -> Net-(J3-S)
- R5 pad 2: Net-(U1-GPIO9) -> Net-(U1-GPIO18/USBD_-)
- U1 pad 12: Net-(U1-GPIO9) -> unconnected-(U1-GPIO9-Pad12)
- U1 pad 18: Net-(U1-GPIO19/USBD_+) -> unconnected-(U1-GPIO19/USBD_+-Pad18)
- U1 pad 19: unconnected-(U1-GPIO18/USBD_--Pad19) -> Net-(U1-GPIO18/USBD_-)
- U1 pad 26: GND -> Net-(J3-S)
Routing:
- net Net-(J3-S): track 0.00 -> 83.0 mm
- net Net-(U1-GPIO9): track 63.1 -> 0.00 mm
- net Net-(U1-GPIO18/USBD_-): track 0.00 -> 40.6 mm
- net Net-(U1-GPIO19/USBD_+): track 26.4 -> 0.00 mm
- net Net-(R10-Pad1): track 14.4 -> 0.00 mm
- net GND: track 367.6 -> 358.7 mm
- net unconnected-(U1-GPIO19/USBD_+-Pad18): track 0.00 -> 1.03 mm
- net 5V: track 397.1 -> 396.2 mm
